File: pcb/ABIMC Board.brd (EAGLE design)
At the start: 81.9 x 48.9 mm, 17 parts

Commit message: Big update!
Revamped the tests, showing the progression of the development.
Updates to the PCB, including getting the clock and data pins in the right order.
Moved some stuff to lib directory (Need to create issue to modularize these)

Known bugs (Need to create issues for these):
When hand moves into new pixel, the pixel sometimes flashes.
Complete power cycle loses connection to GPS.  Reset fixes.
Hands reset early and sometimes jump around.
Parts:
- moved POWER 0.64 mm to (5.08, 17.8)
Connections:
- removed net DSCLOCK1: JP1.3, LS1.3
- removed net DSCLOCK2: JP2.3, LS1.11
- removed net DSCLOCK3: JP3.3, LS1.8
- removed net DSCLOCK4: JP4.3, LS2.11
- removed net DSCLOCK5: JP5.3, LS2.8
- removed net DSCLOCK6: JP6.3, LS2.6
- new net N$1: JP1.2, LS1.3
- new net N$2: JP2.2, LS1.11
- new net N$3: JP4.2, LS2.11
- new net N$4: JP5.2, LS2.8
- new net N$5: JP6.2, LS2.6
- new net N$6: JP3.2, LS1.8
- net DSDATA: now also JP1.3, JP2.3, JP3.3, JP4.3, JP5.3, JP6.3; no longer JP1.2, JP2.2, JP3.2, JP4.2, JP5.2, JP6.2
Routing:
- net DSCLOCK6: track 36.7 -> 0.00 mm
- net N$5: track 0.00 -> 34.9 mm
- net DSDATA: track 132.9 -> 105.0 mm
- net DSCLOCK3: track 17.6 -> 0.00 mm
- net DSCLOCK5: track 16.9 -> 0.00 mm
- net N$6: track 0.00 -> 15.8 mm
- net N$4: track 0.00 -> 14.8 mm
- net N$1: track 0.00 -> 13.0 mm
- net DSCLOCK2: track 12.2 -> 0.00 mm
- net DSCLOCK1: track 12.0 -> 0.00 mm
- net DSCLOCK4: track 12.0 -> 0.00 mm
- net N$2: track 0.00 -> 10.1 mm
- net N$3: track 0.00 -> 9.42 mm
- net GND: track 188.0 -> 185.8 mm
Other:
- board text added: "Analog Binary Infinity Mirror Clock v1.4"
- board text removed: "Analog Binary Infinity Mirror Clock v1.3"
