File: pcb/ABIMC Board.sch (EAGLE design)
At the start: 17 parts

Commit message: Big update!
Revamped the tests, showing the progression of the development.
Updates to the PCB, including getting the clock and data pins in the right order.
Moved some stuff to lib directory (Need to create issue to modularize these)

Known bugs (Need to create issues for these):
When hand moves into new pixel, the pixel sometimes flashes.
Complete power cycle loses connection to GPS.  Reset fixes.
Hands reset early and sometimes jump around.
Connections:
- removed net DSCLOCK1: JP1.3, LS1A.O
- removed net DSCLOCK2: JP2.3, LS1D.O
- removed net DSCLOCK3: JP3.3, LS1C.O
- removed net DSCLOCK4: JP4.3, LS2D.O
- removed net DSCLOCK5: JP5.3, LS2C.O
- removed net DSCLOCK6: JP6.3, LS2B.O
- new net N$1: JP1.2, LS1A.O
- new net N$2: JP2.2, LS1D.O
- new net N$3: JP4.2, LS2D.O
- new net N$4: JP5.2, LS2C.O
- new net N$5: JP6.2, LS2B.O
- new net N$6: JP3.2, LS1C.O
- net DSDATA: now also JP1.3, JP2.3, JP3.3, JP4.3, JP5.3, JP6.3; no longer JP1.2, JP2.2, JP3.2, JP4.2, JP5.2, JP6.2
Other:
- moved on the sheet: LS1A, LS1C, LS1D, LS2B, LS2C, LS2D
